File: orthoCodeCase.kicad_pcb (KiCad board)
At the start: 2 copper layers, 365 x 160 mm, 214 parts, among them J1 AVR-ISP-6, K1:1 KEYSW, K1:10 KEYSW, K1:11 KEYSW, K1:12 KEYSW, K1:13 KEYSW, K1:14 KEYSW, K1:2 KEYSW, K1:3 KEYSW, K1:4 KEYSW, K1:5 KEYSW, K1:6 KEYSW, K1:7 KEYSW, K1:8 KEYSW, K1:9 KEYSW, K2:1 KEYSW, K2:10 KEYSW, K2:11 KEYSW, K2:13 KEYSW, K2:2 KEYSW, K2:3 KEYSW, K2:4 KEYSW, K2:5 KEYSW, K2:6 KEYSW, K2:7 KEYSW, K2:8 KEYSW, K2:9 KEYSW, K3:0 KEYSW, K3:1 KEYSW, K3:10 KEYSW, K3:11 KEYSW, K3:12 KEYSW, K3:13 KEYSW, K3:2 KEYSW, K3:3 KEYSW, K3:4 KEYSW, K3:5 KEYSW, K3:6 KEYSW, K3:7 KEYSW, K3:8 KEYSW, K3:9 KEYSW, K4:0 KEYSW, K4:1 KEYSW, K4:10 KEYSW, K4:11 KEYSW, K4:12 KEYSW, K4:13 KEYSW, K4:14 KEYSW, K4:2 KEYSW, K4:3 KEYSW, K4:4 KEYSW, K4:5 KEYSW, K4:6 KEYSW, K4:7 KEYSW, K4:8 KEYSW, K4:9 KEYSW, K5:0 KEYSW, K5:1 KEYSW, K5:10 KEYSW, K5:11 KEYSW, K5:12 KEYSW, K5:13 KEYSW, K5:14 KEYSW, K5:2 KEYSW, K5:3 KEYSW, K5:4 KEYSW, K5:5 KEYSW, K5:6 KEYSW, K5:7 KEYSW, K5:8 KEYSW, K5:9 KEYSW, U1 ATmega32A-PU, Y1 Crystal

Commit message: increased size of resistor footprints, new plate design
Parts:
- removed BOOT1: BOOT, cftkb:SW_PUSH_6mm
- removed C1, C2: 22p, cftkb:C_Disc_D3.0mm_W1.6mm_P2.50mm
- removed C3, C4: 0.1u, cftkb:C_Disc_D4.3mm_W1.9mm_P5.00mm
- removed C5: 4.7u, cftkb:CP_Radial_D4.0mm_P1.50mm
- removed D1, D2: 3.6V, cftkb:D_DO-35_SOD27_P5.08mm_Horizontal
- removed D1:1, D1:10, D1:11, D1:12, D1:13, D1:14, D1:2, D1:3, D1:4, D1:5, D1:6, D1:7, D1:8, D1:9, D2:1, D2:10, D2:11, D2:13, D2:2, D2:3, D2:4, D2:5, D2:6, D2:7, D2:8, D2:9, D3:0, D3:1, D3:10, D3:11, D3:12, D3:13, D3:2, D3:3, D3:4, D3:5, D3:6, D3:7, D3:8, D3:9, D4:0, D4:1, D4:10, D4:11, D4:12, D4:13, D4:14, D4:2, D4:3, D4:4, D4:5, D4:6, D4:7, D4:8, D4:9, D5:0, D5:1, D5:10, D5:11, D5:12, D5:13, D5:14, D5:2, D5:3, D5:4, D5:5, D5:6, D5:7, D5:8, D5:9, DVol1: 1N4148, cftkb:D_DO-35_SOD27_P5.08mm_Horizontal
- removed F1: 500mA, cftkb:polyfuse_5.1mm
- removed J1: AVR-ISP-6, cftkb:AVR_ICSP_3x2
- removed K1:1, K1:10, K1:11, K1:2, K1:3, K1:4, K1:9: KEYSW, keebs:Mx_Alps_125
- removed K1:12, K1:13, K1:14, K2:10, K2:11, K2:13, K2:2, K2:3, K2:4, K2:5, K2:6, K2:7, K2:8, K2:9, K3:0, K3:10, K3:11, K3:12, K3:2, K3:3, K3:4, K3:5, K3:6, K3:7, K3:8, K3:9, K4:0, K4:10, K4:11, K4:13, K4:14, K4:2, K4:3, K4:4, K4:5, K4:6, K4:7, K4:8, K4:9, K5:0, K5:1, K5:10, K5:11, K5:12, K5:13, K5:14, K5:2, K5:3, K5:4, K5:5, K5:6, K5:7, K5:8, K5:9: KEYSW, keebs:Mx_Alps_100
- removed K1:5, K1:8: KEYSW, keebs:Mx_Alps_275
- removed K1:6, K1:7, K2:1, K3:13: KEYSW, keebs:Mx_Alps_225
- removed K3:1: KEYSW, keebs:Mx_Alps_175
- removed K4:1, K4:12: KEYSW, keebs:Mx_Alps_150
- removed LED1: POWER, cftkb:LED_D3.0mm
- removed R1, R2: 5.1k, cftkb:R_Axial_DIN0204_L3.6mm_D1.6mm_P7.62mm_Horizontal
- removed R3, R4: 75R, cftkb:R_Axial_DIN0204_L3.6mm_D1.6mm_P7.62mm_Horizontal
- removed R5, R6: 1.5k, cftkb:R_Axial_DIN0204_L3.6mm_D1.6mm_P7.62mm_Horizontal
- removed R7: 10k, cftkb:R_Axial_DIN0204_L3.6mm_D1.6mm_P7.62mm_Horizontal
- removed the REF** at (325.0, 145.0) (x3)
- removed the REF** at (225.0, 95.0) (x2)
- removed the REF** at (220.0, 45.0) (x2)
- removed the REF** at (380.0, 45.0) (x2)
- removed the REF** at (375.0, 130.0) (x2)
- removed the REF** at (300.0, 160.0) (x2)
- removed the REF** at (242.5, 200.0) (x2)
- removed the REF** at (162.5, 200.0) (x2)
- removed the REF** at (115.0, 160.0) (x2)
- removed the REF** at (40.0, 160.0) (x2)
- removed the REF** at (202.5, 145.0) (x2)
- removed the REF** at (40.0, 30.0) (x2)
- removed the REF** at (115.0, 30.0) (x2)
- removed the REF** at (185.0, 30.0) (x2)
- removed the REF** at (220.0, 30.0)
- removed the REF** at (300.0, 30.0) (x2)
- removed the REF** at (370.0, 30.0) (x2)
- removed the REF** at (375.0, 160.0) (x2)
- removed the REF** at (202.5, 172.5) (x2)
- removed the REF** at (180.0, 95.0) (x2)
- removed the REF** at (185.0, 45.0) (x2)
- removed the REF** at (60.0, 45.0) (x2)
- removed the REF** at (125.0, 145.0) (x2)
- removed the REF** at (35.0, 145.0) (x2)
- removed RESET1: RESET, cftkb:SW_PUSH_6mm
- removed RGB1: Breakout Pins, digikey-footprints:PinHeader_1x3_P2.54_Drill1.1mm
- removed SVol1: PEC11R-4215F-S0024, digikey-footprints:Rotary_Encoder_Switched_PEC11R
- removed U1: ATmega32A-PU, cftkb:DIP-40_W15.24mm
- removed USB1: USB4085-GF-A_REVA, USB4085-GF-A_REVA:GCT_USB4085-GF-A_REVA
- removed Y1: Crystal, cftkb:Crystal_HC49-4H_Vertical
- added REF**: standoff hole, standoff hole, F.Cu at (100.0, 162.5)
- added REF**: standoff hole, standoff hole, F.Cu at (20.0, 27.5)
- added REF**: MountingHole_2.2mm_M2_Pad, cftkb:MountingHole_2.2mm_M2_Pad, F.Cu at (300.0, 160.0)
- added REF**: MountingHole_2.2mm_M2_Pad, cftkb:MountingHole_2.2mm_M2_Pad, F.Cu at (375.0, 160.0)
- added REF**: MountingHole_2.2mm_M2_Pad, cftkb:MountingHole_2.2mm_M2_Pad, F.Cu at (370.0, 30.0)
- added REF**: MountingHole_2.2mm_M2_Pad, cftkb:MountingHole_2.2mm_M2_Pad, F.Cu at (300.0, 30.0)
- added REF**: MountingHole_2.2mm_M2_Pad, cftkb:MountingHole_2.2mm_M2_Pad, F.Cu at (242.5, 200.0)
- added REF**: MountingHole_2.2mm_M2_Pad, cftkb:MountingHole_2.2mm_M2_Pad, F.Cu at (162.5, 200.0)
- added REF**: MountingHole_2.2mm_M2_Pad, cftkb:MountingHole_2.2mm_M2_Pad, F.Cu at (115.0, 160.0)
- added REF**: MountingHole_2.2mm_M2_Pad, cftkb:MountingHole_2.2mm_M2_Pad, F.Cu at (40.0, 160.0)
- added REF**: MountingHole_2.2mm_M2_Pad, cftkb:MountingHole_2.2mm_M2_Pad, F.Cu at (40.0, 30.0)
- added REF**: standoff hole, standoff hole, F.Cu at (315.0, 162.5)
- added REF**: MountingHole_2.2mm_M2_Pad, cftkb:MountingHole_2.2mm_M2_Pad, F.Cu at (115.0, 30.0)
- added REF**: MountingHole_2.2mm_M2_Pad, cftkb:MountingHole_2.2mm_M2_Pad, F.Cu at (185.0, 30.0)
- added REF**: standoff hole, standoff hole, F.Cu at (255.0, 27.5)
- added REF**: standoff hole, standoff hole, F.Cu at (150.0, 27.5)
- added REF**: standoff hole, standoff hole, F.Cu at (395.0, 27.5)
- added REF**: standoff hole, standoff hole, F.Cu at (395.0, 162.5)
- added REF**: standoff hole, standoff hole, F.Cu at (227.5, 202.5)
- added REF**: standoff hole, standoff hole, F.Cu at (177.5, 202.5)
- added REF**: standoff hole, standoff hole, F.Cu at (20.0, 162.5)
Routing:
- net Row2: track 316.7 -> 0.00 mm, vias 4 -> 0
- net Row1: track 313.6 -> 0.00 mm, vias 3 -> 0
- net Row4: track 310.8 -> 0.00 mm, vias 1 -> 0
- net Col0: track 310.0 -> 0.00 mm
- net Row5: track 309.7 -> 0.00 mm, vias 1 -> 0
- net Row3: track 294.0 -> 0.00 mm, vias 2 -> 0
- net Col1: track 278.1 -> 0.00 mm
- net +5V: track 272.3 -> 0.00 mm, vias 1 -> 0
- net Col14: track 247.5 -> 0.00 mm
- net Col2: track 242.4 -> 0.00 mm
- net Col13: track 228.3 -> 0.00 mm
- net Col3: track 215.9 -> 0.00 mm
- net Col12: track 212.6 -> 0.00 mm
- net ChannelA: track 201.7 -> 0.00 mm, vias 1 -> 0
- net Col5: track 199.1 -> 0.00 mm
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
Commit message: Plate sent to laser cutters
Parts:
- removed the REF** at (100.0, 162.5)
- removed the REF** at (20.0, 27.5)
- removed the REF** at (300.0, 160.0)
- removed the REF** at (375.0, 160.0)
- removed the REF** at (370.0, 30.0)
- removed the REF** at (300.0, 30.0)
- removed the REF** at (242.5, 200.0)
- removed the REF** at (162.5, 200.0)
- removed the REF** at (115.0, 160.0)
- removed the REF** at (40.0, 160.0)
- removed the REF** at (40.0, 30.0)
- removed the REF** at (315.0, 162.5)
- removed the REF** at (115.0, 30.0)
- removed the REF** at (185.0, 30.0)
- removed the REF** at (255.0, 27.5)
- removed the REF** at (150.0, 27.5)
- removed the REF** at (395.0, 27.5)
- removed the REF** at (395.0, 162.5)
- removed the REF** at (227.5, 202.5)
- removed the REF** at (177.5, 202.5)
- removed the REF** at (20.0, 162.5)
- added BOOT1: BOOT, cftkb:SW_PUSH_6mm, F.Cu at (200.0, 134.5)
- added C1: 22p, cftkb:C_Disc_D3.0mm_W1.6mm_P2.50mm, F.Cu at (191.8, 105.6)
- added C2: 22p, cftkb:C_Disc_D3.0mm_W1.6mm_P2.50mm, F.Cu at (191.8, 100.6)
- added C3: 0.1u, cftkb:C_Disc_D4.3mm_W1.9mm_P5.00mm, F.Cu at (214.5, 99.5)
- added C4: 0.1u, cftkb:C_Disc_D4.3mm_W1.9mm_P5.00mm, F.Cu at (192.8, 95.2)
- added C5: 4.7u, cftkb:CP_Radial_D4.0mm_P1.50mm, F.Cu at (202.5, 55.0)
- added D1: 3.6V, cftkb:D_DO-35_SOD27_P5.08mm_Horizontal, F.Cu at (201.0, 50.0)
- added D1:1: 1N4148, cftkb:D_DO-35_SOD27_P5.08mm_Horizontal, F.Cu at (102.0, 39.5)
- added D1:10: 1N4148, cftkb:D_DO-35_SOD27_P5.08mm_Horizontal, F.Cu at (285.0, 44.0)
- added D1:11: 1N4148, cftkb:D_DO-35_SOD27_P5.08mm_Horizontal, F.Cu at (288.0, 39.5)
- added D1:12: 1N4148, cftkb:D_DO-35_SOD27_P5.08mm_Horizontal, F.Cu at (303.0, 41.0)
- added D1:13: 1N4148, cftkb:D_DO-35_SOD27_P5.08mm_Horizontal, F.Cu at (315.0, 41.5)
- added D1:14: 1N4148, cftkb:D_DO-35_SOD27_P5.08mm_Horizontal, F.Cu at (336.0, 40.0)
- added D1:2: 1N4148, cftkb:D_DO-35_SOD27_P5.08mm_Horizontal, F.Cu at (117.0, 41.0)
- added D1:3: 1N4148, cftkb:D_DO-35_SOD27_P5.08mm_Horizontal, F.Cu at (132.0, 42.5)
- added D1:4: 1N4148, cftkb:D_DO-35_SOD27_P5.08mm_Horizontal, F.Cu at (147.0, 44.0)
- added D1:5: 1N4148, cftkb:D_DO-35_SOD27_P5.08mm_Horizontal, F.Cu at (162.0, 39.5)
- added D1:6: 1N4148, cftkb:D_DO-35_SOD27_P5.08mm_Horizontal, F.Cu at (177.0, 41.0)
- added D1:7: 1N4148, cftkb:D_DO-35_SOD27_P5.08mm_Horizontal, F.Cu at (240.0, 39.5)
- added D1:8: 1N4148, cftkb:D_DO-35_SOD27_P5.08mm_Horizontal, F.Cu at (255.0, 41.0)
- added D1:9: 1N4148, cftkb:D_DO-35_SOD27_P5.08mm_Horizontal, F.Cu at (270.0, 42.5)
- added D2: 3.6V, cftkb:D_DO-35_SOD27_P5.08mm_Horizontal, F.Cu at (199.5, 50.0)
- added D2:1: 1N4148, cftkb:D_DO-35_SOD27_P5.08mm_Horizontal, F.Cu at (99.0, 44.0)
- added D2:10: 1N4148, cftkb:D_DO-35_SOD27_P5.08mm_Horizontal, F.Cu at (282.0, 42.5)
- added D2:11: 1N4148, cftkb:D_DO-35_SOD27_P5.08mm_Horizontal, F.Cu at (291.0, 41.0)
- added D2:13: 1N4148, cftkb:D_DO-35_SOD27_P5.08mm_Horizontal, F.Cu at (318.0, 43.0)
- added D2:2: 1N4148, cftkb:D_DO-35_SOD27_P5.08mm_Horizontal, F.Cu at (114.0, 39.5)
- added D2:3: 1N4148, cftkb:D_DO-35_SOD27_P5.08mm_Horizontal, F.Cu at (129.0, 41.0)
- added D2:4: 1N4148, cftkb:D_DO-35_SOD27_P5.08mm_Horizontal, F.Cu at (144.0, 42.5)
- added D2:5: 1N4148, cftkb:D_DO-35_SOD27_P5.08mm_Horizontal, F.Cu at (159.0, 44.0)
- added D2:6: 1N4148, cftkb:D_DO-35_SOD27_P5.08mm_Horizontal, F.Cu at (174.0, 39.5)
- added D2:7: 1N4148, cftkb:D_DO-35_SOD27_P5.08mm_Horizontal, F.Cu at (237.0, 44.0)
- added D2:8: 1N4148, cftkb:D_DO-35_SOD27_P5.08mm_Horizontal, F.Cu at (252.0, 39.5)
- added D2:9: 1N4148, cftkb:D_DO-35_SOD27_P5.08mm_Horizontal, F.Cu at (267.0, 41.0)
- added D3:0: 1N4148, cftkb:D_DO-35_SOD27_P5.08mm_Horizontal, F.Cu at (87.0, 44.0)
- added D3:1: 1N4148, cftkb:D_DO-35_SOD27_P5.08mm_Horizontal, F.Cu at (96.0, 42.5)
- added D3:10: 1N4148, cftkb:D_DO-35_SOD27_P5.08mm_Horizontal, F.Cu at (279.0, 41.0)
- added D3:11: 1N4148, cftkb:D_DO-35_SOD27_P5.08mm_Horizontal, F.Cu at (294.0, 43.0)
- added D3:12: 1N4148, cftkb:D_DO-35_SOD27_P5.08mm_Horizontal, F.Cu at (306.0, 42.5)
- added D3:13: 1N4148, cftkb:D_DO-35_SOD27_P5.08mm_Horizontal, F.Cu at (321.0, 44.5)
- added D3:2: 1N4148, cftkb:D_DO-35_SOD27_P5.08mm_Horizontal, F.Cu at (111.0, 44.0)
- added D3:3: 1N4148, cftkb:D_DO-35_SOD27_P5.08mm_Horizontal, F.Cu at (126.0, 39.5)
- added D3:4: 1N4148, cftkb:D_DO-35_SOD27_P5.08mm_Horizontal, F.Cu at (141.0, 41.0)
- added D3:5: 1N4148, cftkb:D_DO-35_SOD27_P5.08mm_Horizontal, F.Cu at (156.0, 42.5)
- added D3:6: 1N4148, cftkb:D_DO-35_SOD27_P5.08mm_Horizontal, F.Cu at (171.0, 44.0)
- added D3:7: 1N4148, cftkb:D_DO-35_SOD27_P5.08mm_Horizontal, F.Cu at (234.0, 42.5)
- added D3:8: 1N4148, cftkb:D_DO-35_SOD27_P5.08mm_Horizontal, F.Cu at (249.0, 44.0)
- added D3:9: 1N4148, cftkb:D_DO-35_SOD27_P5.08mm_Horizontal, F.Cu at (264.0, 39.5)
- added D4:0: 1N4148, cftkb:D_DO-35_SOD27_P5.08mm_Horizontal, F.Cu at (84.0, 42.5)
- added D4:1: 1N4148, cftkb:D_DO-35_SOD27_P5.08mm_Horizontal, F.Cu at (93.0, 41.0)
- added D4:10: 1N4148, cftkb:D_DO-35_SOD27_P5.08mm_Horizontal, F.Cu at (276.0, 39.5)
- added D4:11: 1N4148, cftkb:D_DO-35_SOD27_P5.08mm_Horizontal, F.Cu at (297.0, 44.5)
- added D4:12: 1N4148, cftkb:D_DO-35_SOD27_P5.08mm_Horizontal, F.Cu at (309.0, 44.0)
- added D4:13: 1N4148, cftkb:D_DO-35_SOD27_P5.08mm_Horizontal, F.Cu at (327.0, 41.5)
- added D4:14: 1N4148, cftkb:D_DO-35_SOD27_P5.08mm_Horizontal, F.Cu at (333.0, 44.5)
- added D4:2: 1N4148, cftkb:D_DO-35_SOD27_P5.08mm_Horizontal, F.Cu at (108.0, 42.5)
- added D4:3: 1N4148, cftkb:D_DO-35_SOD27_P5.08mm_Horizontal, F.Cu at (123.0, 44.0)
- added D4:4: 1N4148, cftkb:D_DO-35_SOD27_P5.08mm_Horizontal, F.Cu at (138.0, 39.5)
- added D4:5: 1N4148, cftkb:D_DO-35_SOD27_P5.08mm_Horizontal, F.Cu at (153.0, 41.0)
- added D4:6: 1N4148, cftkb:D_DO-35_SOD27_P5.08mm_Horizontal, F.Cu at (168.0, 42.5)
- added D4:7: 1N4148, cftkb:D_DO-35_SOD27_P5.08mm_Horizontal, F.Cu at (231.0, 41.0)
- added D4:8: 1N4148, cftkb:D_DO-35_SOD27_P5.08mm_Horizontal, F.Cu at (246.0, 42.5)
- added D4:9: 1N4148, cftkb:D_DO-35_SOD27_P5.08mm_Horizontal, F.Cu at (261.0, 44.0)
- added D5:0: 1N4148, cftkb:D_DO-35_SOD27_P5.08mm_Horizontal, F.Cu at (81.0, 41.0)
- added D5:1: 1N4148, cftkb:D_DO-35_SOD27_P5.08mm_Horizontal, F.Cu at (90.0, 39.5)
- added D5:10: 1N4148, cftkb:D_DO-35_SOD27_P5.08mm_Horizontal, F.Cu at (273.0, 44.0)
- added D5:11: 1N4148, cftkb:D_DO-35_SOD27_P5.08mm_Horizontal, F.Cu at (300.0, 39.5)
- added D5:12: 1N4148, cftkb:D_DO-35_SOD27_P5.08mm_Horizontal, F.Cu at (312.0, 40.0)
- added D5:13: 1N4148, cftkb:D_DO-35_SOD27_P5.08mm_Horizontal, F.Cu at (324.0, 40.0)
- added D5:14: 1N4148, cftkb:D_DO-35_SOD27_P5.08mm_Horizontal, F.Cu at (330.0, 43.0)
- added D5:2: 1N4148, cftkb:D_DO-35_SOD27_P5.08mm_Horizontal, F.Cu at (105.0, 41.0)
- added D5:3: 1N4148, cftkb:D_DO-35_SOD27_P5.08mm_Horizontal, F.Cu at (120.0, 42.5)
- added D5:4: 1N4148, cftkb:D_DO-35_SOD27_P5.08mm_Horizontal, F.Cu at (135.0, 44.0)
- added D5:5: 1N4148, cftkb:D_DO-35_SOD27_P5.08mm_Horizontal, F.Cu at (150.0, 39.5)
- added D5:6: 1N4148, cftkb:D_DO-35_SOD27_P5.08mm_Horizontal, F.Cu at (165.0, 41.0)
- added D5:7: 1N4148, cftkb:D_DO-35_SOD27_P5.08mm_Horizontal, F.Cu at (228.0, 39.5)
- added D5:8: 1N4148, cftkb:D_DO-35_SOD27_P5.08mm_Horizontal, F.Cu at (243.0, 41.0)
- added D5:9: 1N4148, cftkb:D_DO-35_SOD27_P5.08mm_Horizontal, F.Cu at (258.0, 42.5)
- added DVol1: 1N4148, cftkb:D_DO-35_SOD27_P5.08mm_Horizontal, F.Cu at (78.0, 39.5)
- added F1: 500mA, cftkb:polyfuse_5.1mm, F.Cu at (189.5, 55.0)
- added J1: AVR-ISP-6, cftkb:AVR_ICSP_3x2, F.Cu at (187.5, 66.5)
- added K1:1: KEYSW, keebs:Mx_Alps_125, F.Cu at (61.9, 142.9)
- added K1:10: KEYSW, keebs:Mx_Alps_125, F.Cu at (285.8, 142.9)
- added K1:11: KEYSW, keebs:Mx_Alps_125, F.Cu at (309.6, 142.9)
- added K1:12: KEYSW, keebs:Mx_Alps_100, F.Cu at (340.5, 142.9)
- added K1:13: KEYSW, keebs:Mx_Alps_100, F.Cu at (359.6, 142.9)
- added K1:14: KEYSW, keebs:Mx_Alps_100, F.Cu at (378.6, 142.9)
- added K1:2: KEYSW, keebs:Mx_Alps_125, F.Cu at (85.7, 142.9)
- added K1:3: KEYSW, keebs:Mx_Alps_125, F.Cu at (109.5, 142.9)
- added K1:4: KEYSW, keebs:Mx_Alps_125, F.Cu at (142.9, 142.9)
- added K1:5: KEYSW, keebs:Mx_Alps_275, F.Cu at (166.7, 164.3)
- added K1:6: KEYSW, keebs:Mx_Alps_225, F.Cu at (185.7, 169.1)
- added K1:7: KEYSW, keebs:Mx_Alps_225, F.Cu at (219.1, 169.1)
- added K1:8: KEYSW, keebs:Mx_Alps_275, F.Cu at (238.1, 164.3)
- added K1:9: KEYSW, keebs:Mx_Alps_125, F.Cu at (261.9, 142.9)
- added K2:1: KEYSW, keebs:Mx_Alps_225, F.Cu at (61.9, 123.8)
- added K2:10: KEYSW, keebs:Mx_Alps_100, F.Cu at (292.9, 123.8)
- added K2:11: KEYSW, keebs:Mx_Alps_100, F.Cu at (311.9, 123.8)
- added K2:13: KEYSW, keebs:Mx_Alps_100, F.Cu at (359.6, 123.8)
- added K2:2: KEYSW, keebs:Mx_Alps_100, F.Cu at (92.9, 123.8)
- added K2:3: KEYSW, keebs:Mx_Alps_100, F.Cu at (111.9, 123.8)
- added K2:4: KEYSW, keebs:Mx_Alps_100, F.Cu at (131.0, 123.8)
- added K2:5: KEYSW, keebs:Mx_Alps_100, F.Cu at (150.0, 123.8)
- added K2:6: KEYSW, keebs:Mx_Alps_100, F.Cu at (169.1, 123.8)
- added K2:7: KEYSW, keebs:Mx_Alps_100, F.Cu at (235.7, 123.8)
- added K2:8: KEYSW, keebs:Mx_Alps_100, F.Cu at (254.8, 123.8)
- added K2:9: KEYSW, keebs:Mx_Alps_100, F.Cu at (273.8, 123.8)
- added K3:0: KEYSW, keebs:Mx_Alps_100, F.Cu at (35.7, 104.8)
- added K3:1: KEYSW, keebs:Mx_Alps_175, F.Cu at (66.7, 104.8)
- added K3:10: KEYSW, keebs:Mx_Alps_100, F.Cu at (292.9, 104.8)
- added K3:11: KEYSW, keebs:Mx_Alps_100, F.Cu at (311.9, 104.8)
- added K3:12: KEYSW, keebs:Mx_Alps_100, F.Cu at (331.0, 104.8)
- added K3:13: KEYSW, keebs:Mx_Alps_225, F.Cu at (361.9, 104.8)
- added K3:2: KEYSW, keebs:Mx_Alps_100, F.Cu at (92.9, 104.8)
- added K3:3: KEYSW, keebs:Mx_Alps_100, F.Cu at (111.9, 104.8)
- added K3:4: KEYSW, keebs:Mx_Alps_100, F.Cu at (131.0, 104.8)
- added K3:5: KEYSW, keebs:Mx_Alps_100, F.Cu at (150.0, 104.8)
- added K3:6: KEYSW, keebs:Mx_Alps_100, F.Cu at (169.1, 104.8)
- added K3:7: KEYSW, keebs:Mx_Alps_100, F.Cu at (235.7, 104.8)
- added K3:8: KEYSW, keebs:Mx_Alps_100, F.Cu at (254.8, 104.8)
- added K3:9: KEYSW, keebs:Mx_Alps_100, F.Cu at (273.8, 104.8)
- added K4:0: KEYSW, keebs:Mx_Alps_100, F.Cu at (40.5, 85.7)
- added K4:1: KEYSW, keebs:Mx_Alps_150, F.Cu at (69.1, 85.7)
- added K4:10: KEYSW, keebs:Mx_Alps_100, F.Cu at (292.9, 85.7)
- added K4:11: KEYSW, keebs:Mx_Alps_100, F.Cu at (311.9, 85.7)
- added K4:12: KEYSW, keebs:Mx_Alps_150, F.Cu at (335.8, 85.7)
- added K4:13: KEYSW, keebs:Mx_Alps_100, F.Cu at (359.6, 85.7)
- added K4:14: KEYSW, keebs:Mx_Alps_100, F.Cu at (378.6, 85.7)
- added K4:2: KEYSW, keebs:Mx_Alps_100, F.Cu at (92.9, 85.7)
- added K4:3: KEYSW, keebs:Mx_Alps_100, F.Cu at (111.9, 85.7)
- added K4:4: KEYSW, keebs:Mx_Alps_100, F.Cu at (131.0, 85.7)
- added K4:5: KEYSW, keebs:Mx_Alps_100, F.Cu at (150.0, 85.7)
- added K4:6: KEYSW, keebs:Mx_Alps_100, F.Cu at (169.1, 85.7)
- added K4:7: KEYSW, keebs:Mx_Alps_100, F.Cu at (235.7, 85.7)
- added K4:8: KEYSW, keebs:Mx_Alps_100, F.Cu at (254.8, 85.7)
- added K4:9: KEYSW, keebs:Mx_Alps_100, F.Cu at (273.8, 85.7)
- added K5:0: KEYSW, keebs:Mx_Alps_100, F.Cu at (45.2, 66.7)
- added K5:1: KEYSW, keebs:Mx_Alps_100, F.Cu at (69.1, 66.7)
- added K5:10: KEYSW, keebs:Mx_Alps_100, F.Cu at (292.9, 66.7)
- added K5:11: KEYSW, keebs:Mx_Alps_100, F.Cu at (311.9, 66.7)
- added K5:12: KEYSW, keebs:Mx_Alps_100, F.Cu at (331.0, 66.7)
- added K5:13: KEYSW, keebs:Mx_Alps_100, F.Cu at (350.0, 66.7)
- added K5:14: KEYSW, keebs:Mx_Alps_100, F.Cu at (369.1, 66.7)
- added K5:2: KEYSW, keebs:Mx_Alps_100, F.Cu at (92.9, 66.7)
- added K5:3: KEYSW, keebs:Mx_Alps_100, F.Cu at (111.9, 66.7)
- added K5:4: KEYSW, keebs:Mx_Alps_100, F.Cu at (131.0, 66.7)
- added K5:5: KEYSW, keebs:Mx_Alps_100, F.Cu at (150.0, 66.7)
- added K5:6: KEYSW, keebs:Mx_Alps_100, F.Cu at (169.1, 66.7)
- added K5:7: KEYSW, keebs:Mx_Alps_100, F.Cu at (235.7, 66.7)
- added K5:8: KEYSW, keebs:Mx_Alps_100, F.Cu at (254.8, 66.7)
- added K5:9: KEYSW, keebs:Mx_Alps_100, F.Cu at (273.8, 66.7)
- added LED1: POWER, cftkb:LED_D3.0mm, F.Cu at (214.4, 60.0)
- added R1: 5.1k, cftkb:R_Axial_DIN0204_L3.6mm_D1.6mm_P7.62mm_Horizontal, F.Cu at (205.5, 68.0)
- added R2: 5.1k, cftkb:R_Axial_DIN0204_L3.6mm_D1.6mm_P7.62mm_Horizontal, F.Cu at (203.0, 68.0)
- added R3: 75R, cftkb:R_Axial_DIN0204_L3.6mm_D1.6mm_P7.62mm_Horizontal, F.Cu at (200.5, 68.0)
- added R4: 75R, cftkb:R_Axial_DIN0204_L3.6mm_D1.6mm_P7.62mm_Horizontal, F.Cu at (198.0, 68.0)
- added R5: 1.5k, cftkb:R_Axial_DIN0204_L3.6mm_D1.6mm_P7.62mm_Horizontal, F.Cu at (195.5, 68.0)
- added R6: 1.5k, cftkb:R_Axial_DIN0204_L3.6mm_D1.6mm_P7.62mm_Horizontal, F.Cu at (208.0, 60.5)
- added R7: 10k, cftkb:R_Axial_DIN0204_L3.6mm_D1.6mm_P7.62mm_Horizontal, F.Cu at (210.5, 60.5)
- added REF** (x3): MountingHole_2.2mm_M2_Pad, cftkb:MountingHole_2.2mm_M2_Pad, F.Cu at (325.0, 145.0)
- added REF** (x2): MountingHole_2.2mm_M2_Pad, cftkb:MountingHole_2.2mm_M2_Pad, F.Cu at (225.0, 95.0)
- added REF** (x2): MountingHole_2.2mm_M2_Pad, cftkb:MountingHole_2.2mm_M2_Pad, F.Cu at (220.0, 45.0)
- added REF** (x2): MountingHole_2.2mm_M2_Pad, cftkb:MountingHole_2.2mm_M2_Pad, F.Cu at (380.0, 45.0)
- added REF** (x2): MountingHole_2.2mm_M2_Pad, cftkb:MountingHole_2.2mm_M2_Pad, F.Cu at (375.0, 130.0)
- added REF** (x2): MountingHole_2.2mm_M2_Pad, cftkb:MountingHole_2.2mm_M2_Pad, F.Cu at (300.0, 160.0)
- added REF** (x2): MountingHole_2.2mm_M2_Pad, cftkb:MountingHole_2.2mm_M2_Pad, F.Cu at (242.5, 200.0)
- added REF** (x2): MountingHole_2.2mm_M2_Pad, cftkb:MountingHole_2.2mm_M2_Pad, F.Cu at (162.5, 200.0)
- added REF** (x2): MountingHole_2.2mm_M2_Pad, cftkb:MountingHole_2.2mm_M2_Pad, F.Cu at (115.0, 160.0)
- added REF** (x2): MountingHole_2.2mm_M2_Pad, cftkb:MountingHole_2.2mm_M2_Pad, F.Cu at (40.0, 160.0)
- added REF** (x2): MountingHole_2.2mm_M2_Pad, cftkb:MountingHole_2.2mm_M2_Pad, F.Cu at (202.5, 145.0)
- added REF** (x2): MountingHole_2.2mm_M2_Pad, cftkb:MountingHole_2.2mm_M2_Pad, F.Cu at (40.0, 30.0)
- added REF** (x2): MountingHole_2.2mm_M2_Pad, cftkb:MountingHole_2.2mm_M2_Pad, F.Cu at (115.0, 30.0)
- added REF** (x2): MountingHole_2.2mm_M2_Pad, cftkb:MountingHole_2.2mm_M2_Pad, F.Cu at (185.0, 30.0)
- added REF**: MountingHole_2.2mm_M2_Pad, cftkb:MountingHole_2.2mm_M2_Pad, F.Cu at (220.0, 30.0)
- added REF** (x2): MountingHole_2.2mm_M2_Pad, cftkb:MountingHole_2.2mm_M2_Pad, F.Cu at (300.0, 30.0)
- added REF** (x2): MountingHole_2.2mm_M2_Pad, cftkb:MountingHole_2.2mm_M2_Pad, F.Cu at (370.0, 30.0)
- added REF** (x2): MountingHole_2.2mm_M2_Pad, cftkb:MountingHole_2.2mm_M2_Pad, F.Cu at (375.0, 160.0)
- added REF** (x2): MountingHole_2.2mm_M2_Pad, cftkb:MountingHole_2.2mm_M2_Pad, F.Cu at (202.5, 172.5)
- added REF** (x2): MountingHole_2.2mm_M2_Pad, cftkb:MountingHole_2.2mm_M2_Pad, F.Cu at (180.0, 95.0)
- added REF** (x2): MountingHole_2.2mm_M2_Pad, cftkb:MountingHole_2.2mm_M2_Pad, F.Cu at (185.0, 45.0)
- added REF** (x2): MountingHole_2.2mm_M2_Pad, cftkb:MountingHole_2.2mm_M2_Pad, F.Cu at (60.0, 45.0)
- added REF** (x2): MountingHole_2.2mm_M2_Pad, cftkb:MountingHole_2.2mm_M2_Pad, F.Cu at (125.0, 145.0)
- added REF** (x2): MountingHole_2.2mm_M2_Pad, cftkb:MountingHole_2.2mm_M2_Pad, F.Cu at (35.0, 145.0)
- added RESET1: RESET, cftkb:SW_PUSH_6mm, F.Cu at (211.0, 134.5)
- added RGB1: Breakout Pins, digikey-footprints:PinHeader_1x3_P2.54_Drill1.1mm, F.Cu at (80.0, 107.2)
- added SVol1: PEC11R-4215F-S0024, digikey-footprints:Rotary_Encoder_Switched_PEC11R, F.Cu at (39.5, 47.5)
- added U1: ATmega32A-PU, cftkb:DIP-40_W15.24mm, F.Cu at (195.3, 73.8)
- added USB1: USB4085-GF-A_REVA, USB4085-GF-A_REVA:GCT_USB4085-GF-A_REVA, F.Cu at (202.5, 37.0)
- added Y1: Crystal, cftkb:Crystal_HC49-4H_Vertical, F.Cu at (187.8, 105.5)
Routing:
- net Row2: track 0.00 -> 316.7 mm, vias 0 -> 4
- net Row1: track 0.00 -> 313.6 mm, vias 0 -> 3
- net Row4: track 0.00 -> 310.8 mm, vias 0 -> 1
- net Col0: track 0.00 -> 310.0 mm
- net Row5: track 0.00 -> 309.7 mm, vias 0 -> 1
- net Row3: track 0.00 -> 294.0 mm, vias 0 -> 2
- net Col1: track 0.00 -> 278.1 mm
- net +5V: track 0.00 -> 272.3 mm, vias 0 -> 1
- net Col14: track 0.00 -> 247.5 mm
- net Col2: track 0.00 -> 242.4 mm
- net Col13: track 0.00 -> 228.3 mm
- net Col3: track 0.00 -> 215.9 mm
- net Col12: track 0.00 -> 212.6 mm
- net ChannelA: track 0.00 -> 201.7 mm, vias 0 -> 1
- net Col5: track 0.00 -> 199.1 mm
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